Commit message: Wait for URDF meshes and fix asset resolution

File: frontend/public/robot/g1/g1.urdf (robot description, URDF)
Before this commit: robot g1, 40 links, 39 joints
Links:
- link head_link: geometry collision mesh filename=assets/collisions/head_link_collision.STL; visual mesh filename=assets/visuals/head_link.STL
- link left_ankle_pitch_link: geometry visual mesh filename=assets/visuals/left_ankle_pitch_link.STL
- link left_ankle_roll_link: geometry collision mesh filename=assets/collisions/left_ankle_roll_link_collision.STL; visual mesh filename=assets/visuals/left_ankle_roll_link.STL
- link left_elbow_link: geometry collision mesh filename=assets/collisions/left_elbow_link_collision.STL; visual mesh filename=assets/visuals/left_elbow_link.STL
- link left_hip_pitch_link: geometry collision mesh filename=assets/collisions/left_hip_pitch_link_collision.STL; visual mesh filename=assets/visuals/left_hip_pitch_link.STL
- link left_hip_roll_link: geometry collision mesh filename=assets/collisions/left_hip_roll_link_collision.STL; visual mesh filename=assets/visuals/left_hip_roll_link.STL
- link left_hip_yaw_link: geometry collision mesh filename=assets/collisions/left_hip_yaw_link_collision.STL; visual mesh filename=assets/visuals/left_hip_yaw_link.STL
- link left_knee_link: geometry collision mesh filename=assets/collisions/left_knee_link_collision.STL; visual mesh filename=assets/visuals/left_knee_link.STL
- link left_rubber_hand: geometry collision mesh filename=assets/collisions/left_wrist_hand_collision.STL; visual mesh filename=assets/visuals/left_rubber_hand.STL
- link left_shoulder_pitch_link: geometry collision mesh filename=assets/collisions/left_shoulder_pitch_link_collision.STL; visual mesh filename=assets/visuals/left_shoulder_pitch_link.STL
- link left_shoulder_roll_link: geometry collision mesh filename=assets/collisions/left_shoulder_roll_link_collision.STL; visual mesh filename=assets/visuals/left_shoulder_roll_link.STL
- link left_shoulder_yaw_link: geometry collision mesh filename=assets/collisions/left_shoulder_yaw_link_collision.STL; visual mesh filename=assets/visuals/left_shoulder_yaw_link.STL
- link left_wrist_pitch_link: geometry collision mesh filename=assets/collisions/left_wrist_pitch_link_collision.STL; visual mesh filename=assets/visuals/left_wrist_pitch_link.STL
- link left_wrist_roll_link: geometry collision mesh filename=assets/collisions/left_wrist_roll_link_collision.STL; visual mesh filename=assets/visuals/left_wrist_roll_link.STL
- link left_wrist_yaw_link: geometry visual mesh filename=assets/visuals/left_wrist_yaw_link.STL
- link logo_link: geometry visual mesh filename=assets/visuals/logo_link.STL
- link pelvis: geometry collision mesh filename=assets/collisions/pelvis_collision.STL; visual mesh filename=assets/visuals/pelvis.STL
- link pelvis_contour_link: geometry visual mesh filename=assets/visuals/pelvis_contour_link.STL
- link right_ankle_pitch_link: geometry visual mesh filename=assets/visuals/right_ankle_pitch_link.STL
- link right_ankle_roll_link: geometry collision mesh filename=assets/collisions/right_ankle_roll_link_collision.STL; visual mesh filename=assets/visuals/right_ankle_roll_link.STL
- link right_elbow_link: geometry collision mesh filename=assets/collisions/right_elbow_link_collision.STL; visual mesh filename=assets/visuals/right_elbow_link.STL
- link right_hip_pitch_link: geometry collision mesh filename=assets/collisions/right_hip_pitch_link_collision.STL; visual mesh filename=assets/visuals/right_hip_pitch_link.STL
- link right_hip_roll_link: geometry collision mesh filename=assets/collisions/right_hip_roll_link_collision.STL; visual mesh filename=assets/visuals/right_hip_roll_link.STL
- link right_hip_yaw_link: geometry collision mesh filename=assets/collisions/right_hip_yaw_link_collision.STL; visual mesh filename=assets/visuals/right_hip_yaw_link.STL
- link right_knee_link: geometry collision mesh filename=assets/collisions/right_knee_link_collision.STL; visual mesh filename=assets/visuals/right_knee_link.STL
- link right_rubber_hand: geometry collision mesh filename=assets/collisions/right_wrist_hand_collision.STL; visual mesh filename=assets/visuals/right_rubber_hand.STL
- link right_shoulder_pitch_link: geometry collision mesh filename=assets/collisions/right_shoulder_pitch_link_collision.STL; visual mesh filename=assets/visuals/right_shoulder_pitch_link.STL
- link right_shoulder_roll_link: geometry collision mesh filename=assets/collisions/right_shoulder_roll_link_collision.STL; visual mesh filename=assets/visuals/right_shoulder_roll_link.STL
- link right_shoulder_yaw_link: geometry collision mesh filename=assets/collisions/right_shoulder_yaw_link_collision.STL; visual mesh filename=assets/visuals/right_shoulder_yaw_link.STL
- link right_wrist_pitch_link: geometry collision mesh filename=assets/collisions/right_wrist_pitch_link_collision.STL; visual mesh filename=assets/visuals/right_wrist_pitch_link.STL
- link right_wrist_roll_link: geometry collision mesh filename=assets/collisions/right_wrist_roll_link_collision.STL; visual mesh filename=assets/visuals/right_wrist_roll_link.STL
- link right_wrist_yaw_link: geometry visual mesh filename=assets/visuals/right_wrist_yaw_link.STL
- link torso_link: geometry collision mesh filename=assets/collisions/torso_waist_roll_pitch_collision.STL; visual mesh filename=assets/visuals/torso_link_rev_1_0.STL
- link waist_roll_link: geometry visual mesh filename=assets/visuals/waist_roll_link_rev_1_0.STL
- link waist_yaw_link: geometry visual mesh filename=assets/visuals/waist_yaw_link_rev_1_0.STL
