Commit message: Inlay FAVL in the G1 chest plate
The mark sits in a recessed plaque on the torso surface instead of
floating in front of the armor. Joint offset is identity so the
mesh is in chest coordinates.

File: frontend/public/robot/g1/g1.urdf (robot description, URDF)
Before this commit: robot g1, 40 links, 39 joints
Links:
- link logo_link: geometry visual mesh filename=assets/visuals/logo_link.STL; visual mesh filename=assets/visuals/logo_plate.STL
Joints:
- joint logo_joint: origin xyz=0.0039635 0 -0.044 rpy=0 0 0 -> xyz=0 0 0 rpy=0 0 0

Commit message: Carve FAVL and a hexagon mic into the chest
Remove the speech bubble. Green is only the FAVL letters while
speaking. A recessed hexagon on the belly starts the microphone
and lights green; standby is neon blue. Right wrist no longer twists.

File: frontend/public/robot/g1/g1.urdf (robot description, URDF)
Before this commit: robot g1, 40 links, 39 joints
Links:
- added link mic_button_link, mass 0.001; visual mesh filename=assets/visuals/mic_button.STL
Joints:
- added joint mic_joint: type fixed, parent torso_link, child mic_button_link, origin xyz=0 0 0 rpy=0 0 0

Commit message: Embed the chest button and let a press ask what to do
Sink the navel into a carved torso well, drop the overlay sticker, and
have the G1 ask demo or sign-in then point you to the next step.

File: frontend/public/robot/g1/g1.urdf (robot description, URDF)
Before this commit: robot g1, 41 links, 40 joints
Links:
- link mic_button_link: geometry visual mesh filename=assets/visuals/mic_button.STL; visual mesh filename=assets/visuals/mic_well.STL
